Commit message: added axis to joints

File: src/urdf/rosrobot-proto1.urdf (robot description, URDF)
Before this commit: robot rosrobot, 8 links, 7 joints
Joints:
- joint base_to_sideplate_left: origin xyz=0 0.07 0 -> xyz=0 0.07 0 rpy=0 0 0
- joint base_to_sideplate_right: origin xyz=0 -0.07 0 -> xyz=0 -0.07 0 rpy=0 0 0
- joint base_to_topbase: origin xyz=0 0 0.03 -> xyz=0 0 0.03 rpy=0 0 0
- joint base_to_wheel_left_back: axis (none) -> 0 1 0; origin xyz=-0.080 0.0865 0 -> xyz=-0.080 0.0865 0 rpy=0 0 0; type fixed -> continuous
- joint base_to_wheel_left_front: axis (none) -> 0 1 0; origin xyz=0.080 0.0865 0 -> xyz=0.080 0.0865 0 rpy=0 0 0; type fixed -> continuous
- joint base_to_wheel_right_back: axis (none) -> 0 1 0; origin xyz=-0.080 -0.0865 0 -> xyz=-0.080 -0.0865 0 rpy=0 0 0; type fixed -> continuous
- joint base_to_wheel_right_front: axis (none) -> 0 1 0; origin xyz=0.080 -0.0865 0 -> xyz=0.080 -0.0865 0 rpy=0 0 0; type fixed -> continuous
